File: Final/ProbeStationRelayBoard.brd (EAGLE design)
At the start: 100 x 100 mm, 47 parts, among them K1 G6DN-1A_DC12, K10 G6DN-1A_DC12, K11 G6DN-1A_DC12, K12 G6DN-1A_DC12, K13 G6DN-1A_DC12, K14 G6DN-1A_DC12, K15 G6DN-1A_DC12, K16 G6DN-1A_DC12, K17 G6DN-1A_DC12, K18 G6DN-1A_DC12, K19 G6DN-1A_DC12, K2 G6DN-1A_DC12, K20 G6DN-1A_DC12, K21 G6DN-1A_DC12, K22 G6DN-1A_DC12, K23 G6DN-1A_DC12, K24 G6DN-1A_DC12, K25 G6DN-1A_DC12, K26 G6DN-1A_DC12, K27 G6DN-1A_DC12, K28 G6DN-1A_DC12, K29 G6DN-1A_DC12, K3 G6DN-1A_DC12, K30 G6DN-1A_DC12, K31 G6DN-1A_DC12, K32 G6DN-1A_DC12, K4 G6DN-1A_DC12, K5 G6DN-1A_DC12, K6 G6DN-1A_DC12, K7 G6DN-1A_DC12, K8 G6DN-1A_DC12, K9 G6DN-1A_DC12, U1 MC14515BDWR2G, U2 MC14515BDWR2G, U3 CD4504BPWR, U4 CD4504BPWR

Commit message: Revise final layout and schematic
Parts:
- added C1, C2, C3, C4, C5, C6: (no value), rcl:C0805
- moved 5VPWR 19.1 mm to (93.0, 22.4)
- moved JP5 4.60 mm to (84.6, 51.3)
- moved JP6 4.44 mm to (84.6, 61.3)
- renumbered SRC0 to SRC2
Connections:
- net GND: now also C1.2, C2.2, C3.2, C4.2, C5.2, C6.2, SRC1.2, SRC1.3, SRC1.4, SRC1.5, SRC2.2, SRC2.3, SRC2.4, SRC2.5
- net SRC1: now also C1.1, C2.1, C3.1
- net SRC2: now also C4.1, C5.1, C6.1
Routing:
- net GND: track 164.7 -> 90.9 mm
- net +5V: track 94.3 -> 110.0 mm
- net SRC1: track 117.2 -> 122.5 mm, vias 0 -> 1
- net SRC2: track 178.0 -> 181.2 mm
- net S0: track 87.4 -> 89.4 mm
- net +12V: track 89.5 -> 91.2 mm
- net S1: track 82.0 -> 80.4 mm
- net S3: track 69.5 -> 68.5 mm
- net INH_C: track 10.2 -> 11.1 mm
- added copper zone on layer 1, net GND
