File: Final/ProbeStationRelayBoard.sch (EAGLE design)
At the start: 47 parts, among them K1 G6DN-1A_DC12, K10 G6DN-1A_DC12, K11 G6DN-1A_DC12, K12 G6DN-1A_DC12, K13 G6DN-1A_DC12, K14 G6DN-1A_DC12, K15 G6DN-1A_DC12, K16 G6DN-1A_DC12, K17 G6DN-1A_DC12, K18 G6DN-1A_DC12, K19 G6DN-1A_DC12, K2 G6DN-1A_DC12, K20 G6DN-1A_DC12, K21 G6DN-1A_DC12, K22 G6DN-1A_DC12, K23 G6DN-1A_DC12, K24 G6DN-1A_DC12, K25 G6DN-1A_DC12, K26 G6DN-1A_DC12, K27 G6DN-1A_DC12, K28 G6DN-1A_DC12, K29 G6DN-1A_DC12, K3 G6DN-1A_DC12, K30 G6DN-1A_DC12, K31 G6DN-1A_DC12, K32 G6DN-1A_DC12, K4 G6DN-1A_DC12, K5 G6DN-1A_DC12, K6 G6DN-1A_DC12, K7 G6DN-1A_DC12, K8 G6DN-1A_DC12, K9 G6DN-1A_DC12, U1 MC14515BDWR2G, U2 MC14515BDWR2G, U3 CD4504BPWR, U4 CD4504BPWR

Commit message: Revise final layout and schematic
Parts:
- removed SRC0: BU-SMA-V, con-coax:BU-SMA-V
- added C1, C2, C3, C4, C5, C6: (no value), rcl:C-USC0805
- added SRC2: BU-SMA-V, con-coax:BU-SMA-V
Connections:
- net GND: now also C1.2, C2.2, C3.2, C4.2, C5.2, C6.2, SRC1.2, SRC2.2
- net SRC1: now also C1.1, C2.1, C3.1
- net SRC2: now also C4.1, C5.1, C6.1, SRC2.1; no longer SRC0.1
Other:
- moved on the sheet: 12VPWR, 5VPWR, JP5, JP6, SRC1, U3, U4
